File: hardware/motors.sch (KiCad schematic (older format))
At the start: 4 parts

Commit message: changes on stream
Parts:
- J3, J4, J5, J6: renamed from J?; footprint (none) -> Connector_PinHeader_2.54mm:PinHeader_1x02_P2.54mm_Horizontal
Changed lines of the file:
@@
 $EndDescr
 $Comp
-L Connector:Conn_01x02_Female J?
+L Connector:Conn_01x02_Female J3
 U 1 1 5E94E945
 P 8150 2900
-F 0 "J?" H 8178 2876 50  0000 L CNN
+F 0 "J3" H 8178 2876 50  0000 L CNN
 F 1 "Motor A" H 8178 2785 50  0000 L CNN
-F 2 "" H 8150 2900 50  0001 C CNN
+F 2 "Connector_PinHeader_2.54mm:PinHeader_1x02_P2.54mm_Horizontal" H 8150 2900 50  0001 C CNN
 F 3 "~" H 8150 2900 50  0001 C CNN
 	1    8150 2900
@@
 $EndComp
 $Comp
-L Connector:Conn_01x02_Female J?
+L Connector:Conn_01x02_Female J4
 U 1 1 5E94E94B
 P 8150 3200
-F 0 "J?" H 8178 3176 50  0000 L CNN
+F 0 "J4" H 8178 3176 50  0000 L CNN
 F 1 "Motor B" H 8178 3085 50  0000 L CNN
-F 2 "" H 8150 3200 50  0001 C CNN
+F 2 "Connector_PinHeader_2.54mm:PinHeader_1x02_P2.54mm_Horizontal" H 8150 3200 50  0001 C CNN
 F 3 "~" H 8150 3200 50  0001 C CNN
 	1    8150 3200
@@
 $EndComp
 $Comp
-L Connector:Conn_01x02_Female J?
+L Connector:Conn_01x02_Female J5
 U 1 1 5E94E951
 P 8150 3500
-F 0 "J?" H 8178 3476 50  0000 L CNN
+F 0 "J5" H 8178 3476 50  0000 L CNN
 F 1 "Motor C" H 8178 3385 50  0000 L CNN
-F 2 "" H 8150 3500 50  0001 C CNN
+F 2 "Connector_PinHeader_2.54mm:PinHeader_1x02_P2.54mm_Horizontal" H 8150 3500 50  0001 C CNN
 F 3 "~" H 8150 3500 50  0001 C CNN
 	1    8150 3500
@@
 $EndComp
 $Comp
-L Connector:Conn_01x02_Female J?
+L Connector:Conn_01x02_Female J6
 U 1 1 5E94E957
 P 8150 3800
-F 0 "J?" H 8178 3776 50  0000 L CNN
+F 0 "J6" H 8178 3776 50  0000 L CNN
 F 1 "Motor D" H 8178 3685 50  0000 L CNN
-F 2 "" H 8150 3800 50  0001 C CNN
+F 2 "Connector_PinHeader_2.54mm:PinHeader_1x02_P2.54mm_Horizontal" H 8150 3800 50  0001 C CNN
 F 3 "~" H 8150 3800 50  0001 C CNN
 	1    8150 3800
 	1    0    0    -1
 $EndComp
+Text HLabel 5500 3500 0    50   Input ~ 0
+MotorAGo
 $EndSCHEMATC
